Commit message: Adds controller nodes. Thruster controller converts body accel to individual thruster commands and Velocity controller converts body velocity to body acceleration using PID

File: pontus_description/models/pontus/components/thrusters.xacro (robot description, xacro)
@@ -6,4 +6,5 @@
     <link name="thruster_${thruster_id}">
       <visual>
+        <origin xyz="0 0 0" rpy="0 ${180*pi/180} 0"/>
         <geometry>
           <mesh filename="${T200_body_mesh}"/>
@@ -28,4 +29,5 @@
       </inertial>
       <visual>
+        <origin xyz="0 0 0" rpy="0 ${180*pi/180} 0"/>
         <geometry>
           <mesh filename="${T200_prop_mesh}"/>

File: pontus_description/models/pontus/pontus.xacro (robot description, xacro)
@@ -42,33 +42,33 @@
   <!-- Back Left Vertical Thruster -->
   <xacro:T200_macro thruster_id="0">
-    <origin xyz="-0.075 -${radius + 0.07} 0" rpy="0 ${180*pi/180} 0" />
+    <origin xyz="-0.075 -${radius + 0.07} 0" rpy="0 0 0" />
   </xacro:T200_macro>
   <!-- Back Right Vertical Thruster -->
   <xacro:T200_macro thruster_id="1">
-    <origin xyz="-0.075 ${radius + 0.07} 0" rpy="0 ${180*pi/180} ${180*pi/180}" />
+    <origin xyz="-0.075 ${radius + 0.07} 0" rpy="0 0 ${180*pi/180}" />
   </xacro:T200_macro>
   <!-- Front Left Vertical Thruster -->
   <xacro:T200_macro thruster_id="2">
-    <origin xyz="0.075 -${radius + 0.07} 0" rpy="0 ${180*pi/180} 0" />
+    <origin xyz="0.075 -${radius + 0.07} 0" rpy="0 0 0" />
   </xacro:T200_macro>
   <!-- Front Right Vertical Thruster -->
   <xacro:T200_macro thruster_id="3">
-    <origin xyz="0.075 ${radius + 0.07} 0" rpy="0 ${180*pi/180} ${180*pi/180}" />
+    <origin xyz="0.075 ${radius + 0.07} 0" rpy="0 0 ${180*pi/180}" />
   </xacro:T200_macro>
   <!-- Back Left Horizontal Thruster -->
   <xacro:T200_macro thruster_id="4">
-    <origin xyz="-0.2 -${radius + 0.15} 0" rpy="0 -${90*pi/180} 0" />
+    <origin xyz="-0.2 -${radius + 0.15} 0" rpy="0 ${90*pi/180} 0" />
   </xacro:T200_macro>
   <!-- Back Right Horizontal Thruster -->
   <xacro:T200_macro thruster_id="5">
-    <origin xyz="-0.2 ${radius + 0.15} 0" rpy="${180*pi/180}  ${90*pi/180} 0" />
+    <origin xyz="-0.2 ${radius + 0.15} 0" rpy="${180*pi/180}  -${90*pi/180} 0" />
   </xacro:T200_macro>
   <!-- Front Left Horizontal Thruster -->
   <xacro:T200_macro thruster_id="6">
-    <origin xyz="0.2 -${radius + 0.15} 0" rpy="0 -${90*pi/180} 0" />
+    <origin xyz="0.2 -${radius + 0.15} 0" rpy="0 ${90*pi/180} 0" />
   </xacro:T200_macro>
   <!-- Front Right Horizontal Thruster -->
   <xacro:T200_macro thruster_id="7">
-    <origin xyz="0.2 ${radius + 0.15} 0" rpy="${180*pi/180}  ${90*pi/180} 0" />
+    <origin xyz="0.2 ${radius + 0.15} 0" rpy="${180*pi/180}  -${90*pi/180} 0" />
   </xacro:T200_macro>
   <!-- Sensors -->
