Commit message: Add semantic map, prequal autonomy, controller changes

File: pontus_description/models/pontus/components/lights.xacro (robot description, xacro)
@@ -19,7 +19,7 @@
             <pose>0 0 0 0 1.57 3.14</pose>
             <attenuation>
-                <range>4</range>
+                <range>10</range>
                 <constant>1</constant>
-                <linear>0.5</linear>
+                <linear>0.12</linear>
                 <quadratic>0.05</quadratic>
             </attenuation>

File: pontus_description/models/pontus/components/sensors.xacro (robot description, xacro)
@@ -14,8 +14,8 @@
       <sensor name="camera_${camera_id}" type="camera">
         <camera>
-          <horizontal_fov>1.20428</horizontal_fov>
+          <horizontal_fov>1.0472</horizontal_fov>
           <image>
-            <width>320</width>
-            <height>240</height>
+            <width>640</width>
+            <height>480</height>
           </image>
           <clip>
@@ -31,5 +31,15 @@
     </gazebo>
   </xacro:macro>
-  <!-- Sonoptix Echo Sonar  -->
+  <!-- DVL  -->
+  <xacro:macro name="dvl_macro" params="dvl_id *origin">
+    <link name="dvl_a50_link"/>
+    <joint name="dvl_joint_${dvl_id}" type="fixed">
+      <xacro:insert_block name="origin"/>
+      <parent link="base_link"/>
+      <child link="dvl_a50_link"/>
+      <axis xyz="1 0 0"/>
+    </joint>
+  </xacro:macro>
+  <!-- Sonoptix Echo  -->
   <xacro:macro name="sonoptix_macro" params="sonar_id *origin">
     <link name="sonar_${sonar_id}">

File: pontus_description/models/pontus/pontus.xacro (robot description, xacro)
@@ -9,5 +9,5 @@
   <xacro:property name="fluid_density" value="1025"/>
   <xacro:property name="namespace" value="pontus"/>
-  <xacro:property name="mass" value="50"/>
+  <xacro:property name="mass" value="34.0194"/>
   <xacro:property name="length" value="0.61"/>
   <xacro:property name="radius" value="0.1"/>
@@ -17,5 +17,5 @@
     <inertial>
       <!-- This is calculated for slightly positive buoyancy -->
-      <mass value="${(volume * fluid_density) - 1.0}"/>
+      <mass value="${(volume * fluid_density) - 5.0}"/>
       <!-- TODO: insert actual calculations instead of precalculated value -->
       <inertia
@@ -59,17 +59,17 @@
   <!-- Back Left Horizontal Thruster -->
   <xacro:T200_macro thruster_id="4">
-    <origin xyz="-0.2 ${radius + 0.15} 0" rpy="${180*pi/180}  -${90*pi/180} 0" />
+    <origin xyz="-0.25 ${radius + 0.15} 0" rpy="${180*pi/180}  -${90*pi/180} ${5/4 * pi}" />
   </xacro:T200_macro>
   <!-- Back Right Horizontal Thruster -->
   <xacro:T200_macro thruster_id="5">
-    <origin xyz="-0.2 -${radius + 0.15} 0" rpy="0 ${90*pi/180} 0" />
+    <origin xyz="-0.25 -${radius + 0.15} 0" rpy="0 ${90*pi/180} ${3/4 * pi}" />
   </xacro:T200_macro>
   <!-- Front Left Horizontal Thruster -->
   <xacro:T200_macro thruster_id="6">
-    <origin xyz="0.2 ${radius + 0.15} 0" rpy="${180*pi/180}  -${90*pi/180} 0" />
+    <origin xyz="0.25 ${radius + 0.15} 0" rpy="${180*pi/180}  -${90*pi/180} ${-1/4 * pi}" />
   </xacro:T200_macro>
   <!-- Front Right Horizontal Thruster -->
   <xacro:T200_macro thruster_id="7">
-    <origin xyz="0.2 -${radius + 0.15} 0" rpy="0 ${90*pi/180} 0" />
+    <origin xyz="0.25 -${radius + 0.15} 0" rpy="0 ${90*pi/180} ${1/4 * pi}" />
   </xacro:T200_macro>
   <xacro:light_macro light_id="0">
@@ -78,6 +78,16 @@
   <!-- Sensors -->
   <!-- Forward Camera -->
-  <xacro:camera_macro camera_id="0">
+  <xacro:camera_macro camera_id="2">
     <origin xyz="0.305 0 0" rpy="0 0 0" />
+  </xacro:camera_macro>
+    <xacro:camera_macro camera_id="3">
+    <origin xyz="0.305 -0.075 0" rpy="0 0 0" />
+  </xacro:camera_macro>
+  <!-- Side Camera -->
+  <xacro:camera_macro camera_id="4">
+    <origin xyz="0 0.06 0.1" rpy="0 0 ${90*pi/180}" />
+  </xacro:camera_macro>
+  <xacro:camera_macro camera_id="5">
+    <origin xyz="0 -0.06 0.1" rpy="0 0 -${90*pi/180}" />
   </xacro:camera_macro>
   <!-- Downward Camera -->
@@ -87,5 +97,5 @@
   <!-- Forward Sonar -->
   <xacro:sonoptix_macro sonar_id="0">
-    <origin xyz="0.28 0 -0.15" rpy="0 ${25*pi/180} 0" />
+    <origin xyz="0.28 0 -0.15" rpy="${pi} ${10*pi/180} 0" />
   </xacro:sonoptix_macro>
   <!-- 360 Top Sonar -->
@@ -93,7 +103,11 @@
     <origin xyz="0 0 ${radius + 0.02}" rpy="0 0 0" />
   </xacro:ping360_macro>
+  <!-- DVL -->
+  <xacro:dvl_macro dvl_id="0">
+    <origin xyz="0 0 0" rpy="3.141 0 0" />
+  </xacro:dvl_macro>
   <!-- IMU -->
   <xacro:imu_macro imu_id="0">
-    <origin xyz="0 0 0" rpy="0 0 0" />
+    <origin xyz="0 0 0" rpy="1.571 0 -1.571" />
   </xacro:imu_macro>
   <!-- Pressure -->
@@ -127,18 +141,17 @@
         <nDotR>0</nDotR>
         <!-- Linear Drag -->
-        <xU>-10</xU>
-        <yV>-10</yV>
-        <zW>-10</zW>
+        <xU>-5</xU>
+        <yV>-5</yV>
+        <zW>-5</zW>
         <kP>-10</kP>
-        <mQ>-10</mQ>
-        <nR>-10</nR>
-        <!-- Quadratic Drag -->
+        <mQ>-5</mQ>
+        <nR>-5</nR>
         <xUabsU>-6.2282</xUabsU>
-        <yVabsV>-601.27</yVabsV>
-        <zWabsW>-601.27</zWabsW>
+        <yVabsV>-60</yVabsV>
+        <zWabsW>-60</zWabsW>
         <kPabsP>-0.1916</kPabsP>
-        <mQabsQ>-632.698957</mQabsQ>
-        <nRabsR>-632.698957</nRabsR>
-    </plugin>
+        <mQabsQ>-63</mQabsQ>
+        <nRabsR>-500</nRabsR>
+      </plugin>
     <!-- Publishes perfect odometry data for testing controllers -->
     <plugin

File: pontus_description/models/pontus/pontus_real.xacro (robot description, xacro)
@@ -9,5 +9,5 @@
   <xacro:property name="fluid_density" value="1025"/>
   <xacro:property name="namespace" value="pontus"/>
-  <xacro:property name="mass" value="155"/>
+  <xacro:property name="mass" value="156"/>
   <xacro:property name="length" value="0.78"/>
   <xacro:property name="radius" value="0.25"/>
@@ -21,6 +21,6 @@
       <!-- TODO: insert actual calculations instead of precalculated value -->
       <inertia
-        ixx="55" ixy="0" ixz="0"
-        iyy="0.585" iyz="0" izz="55"
+        ixx="156" ixy="0" ixz="0"
+        iyy="0.585" iyz="0" izz="156"
       />
     </inertial>
@@ -88,5 +88,5 @@
   <!-- Forward Sonar -->
   <xacro:sonoptix_macro sonar_id="0">
-    <origin xyz="0.28 0 -0.15" rpy="0 ${25*pi/180} 0" />
+    <origin xyz="0.28 0 -0.15" rpy="0 ${10*pi/180} 0" />
   </xacro:sonoptix_macro>
   <!-- 360 Top Sonar -->
@@ -94,4 +94,8 @@
     <origin xyz="0 0 ${radius + 0.02 - 0.1}" rpy="0 0 0" />
   </xacro:ping360_macro>
+  <!-- DVL -->
+  <xacro:dvl_macro dvl_id="0">
+    <origin xyz="0 0 0" rpy="0 0 0" />
+  </xacro:dvl_macro>
   <!-- IMU -->
   <xacro:imu_macro imu_id="0">
@@ -146,4 +150,6 @@
       filename="gz-sim-odometry-publisher-system"
       name="gz::sim::systems::OdometryPublisher">
+      <odom_frame>odom</odom_frame>
+      <robot_base_frame>base_link</robot_base_frame>
       <dimensions>3</dimensions>
     </plugin>

Commit message: Add tech triton model to sim

File: pontus_description/models/pontus/components/lights.xacro (robot description, xacro)
@@ -1,10 +1,9 @@
 <?xml version="1.0"?>
 <robot xmlns:xacro="http://www.ros.org/wiki/xacro">
-    <!-- Light -->
     <xacro:macro name="light_macro" params="light_id *origin">
     <link name="light_${light_id}">
         <visual>
         <geometry>
-            <cylinder radius="0.02" length="0.1"/> <!-- Define a simple shape for visualization -->
+            <cylinder radius="0.02" length="0.1"/>
         </geometry>
         </visual>
@@ -18,15 +17,15 @@
     <gazebo reference="light_${light_id}">
         <light name="light_${light_id}" type="point">
-        <pose>-0.05 0 0 0 1.57 3.14</pose> <!-- Adjust the position and orientation as needed -->
-        <attenuation>
-            <range>4</range> <!-- The range of the light -->
-            <constant>1</constant>
-            <linear>0.5</linear>
-            <quadratic>0.05</quadratic>
-        </attenuation>
-        <cutoff>0.785</cutoff><!-- Light cone angle (in radians) -->
-        <diffuse>1 1 1 1</diffuse> <!-- Color of the light -->
-        <specular>1 1 1 1</specular>
-        <visualize>false</visualize>
+            <pose>0 0 0 0 1.57 3.14</pose>
+            <attenuation>
+                <range>4</range>
+                <constant>1</constant>
+                <linear>0.5</linear>
+                <quadratic>0.05</quadratic>
+            </attenuation>
+            <cutoff>0.785</cutoff>
+            <diffuse>1 1 1 1</diffuse>
+            <specular>1 1 1 1</specular>
+            <visualize>false</visualize>
         </light>
     </gazebo>

File: pontus_description/models/pontus/pontus.xacro (robot description, xacro)
@@ -4,5 +4,5 @@
   <xacro:include filename="$(find pontus_description)/models/pontus/components/sensors.xacro"/>
   <xacro:include filename="$(find pontus_description)/models/pontus/components/lights.xacro"/>
-  <!--<xacro:property name="mesh_file" value="file://$(find pontus_description)/models/pontus/meshes/pontus_body_mesh.STL"/>-->
+  <xacro:property name="mesh_file" value="file://$(find pontus_description)/models/pontus/meshes/tech_triton.STL"/>
   <xacro:arg name="sim" default="false"/>
   <xacro:arg name="static" default="false"/>
@@ -10,6 +10,6 @@
   <xacro:property name="namespace" value="pontus"/>
   <xacro:property name="mass" value="50"/>
-  <xacro:property name="length" value="0.61"/>
-  <xacro:property name="radius" value="0.1"/>
+  <xacro:property name="length" value="0.78"/>
+  <xacro:property name="radius" value="0.25"/>
   <xacro:property name="volume" value="${pi*length*(radius)**2}"/>
   <!-- Create pontus -->
@@ -25,10 +25,10 @@
     </inertial>
     <visual>
-      <origin xyz="0 0 0" rpy="0 ${-90*pi/180} 0"/>
+      <origin xyz="-0.346957 -0.271635 -0.1620155" rpy="1.57 0 1.57"/>
       <geometry>
-        <cylinder length="${length}" radius="${radius}"/>
+        <mesh filename="${mesh_file}" scale="1 1 1"/>
       </geometry>
       <material name="acrylic">
-        <color rgba="0.9 0.9 0.9 0.4"/>
+        <color rgba="0.5 0.5 0.5 0.8"/>
       </material>
     </visual>
@@ -43,41 +43,41 @@
   <!-- Back Left Vertical Thruster -->
   <xacro:T200_macro thruster_id="0">
-    <origin xyz="-0.075 -${radius + 0.07} 0" rpy="0 0 0" />
+    <origin xyz="-0.0775 -0.2 0" rpy="0 0 0" />
   </xacro:T200_macro>
   <!-- Back Right Vertical Thruster -->
   <xacro:T200_macro thruster_id="1">
-    <origin xyz="-0.075 ${radius + 0.07} 0" rpy="0 0 ${180*pi/180}" />
+    <origin xyz="-0.0775 0.2 0" rpy="0 0 ${180*pi/180}" />
   </xacro:T200_macro>
   <!-- Front Left Vertical Thruster -->
   <xacro:T200_macro thruster_id="2">
-    <origin xyz="0.075 -${radius + 0.07} 0" rpy="0 0 0" />
+    <origin xyz="0.0775 -0.2 0" rpy="0 0 0" />
   </xacro:T200_macro>
   <!-- Front Right Vertical Thruster -->
   <xacro:T200_macro thruster_id="3">
-    <origin xyz="0.075 ${radius + 0.07} 0" rpy="0 0 ${180*pi/180}" />
+    <origin xyz="0.0775 0.2 0" rpy="0 0 ${180*pi/180}" />
   </xacro:T200_macro>
   <!-- Back Left Horizontal Thruster -->
   <xacro:T200_macro thruster_id="4">
-    <origin xyz="-0.2 ${radius + 0.15} 0" rpy="${180*pi/180}  -${90*pi/180} 0" />
+    <origin xyz="-0.2295 0.31 0" rpy="${180*pi/180}  -${90*pi/180} 0" />
   </xacro:T200_macro>
   <!-- Back Right Horizontal Thruster -->
   <xacro:T200_macro thruster_id="5">
-    <origin xyz="-0.2 -${radius + 0.15} 0" rpy="0 ${90*pi/180} 0" />
+    <origin xyz="-0.2295 -0.31 0" rpy="0 ${90*pi/180} 0" />
   </xacro:T200_macro>
   <!-- Front Left Horizontal Thruster -->
   <xacro:T200_macro thruster_id="6">
-    <origin xyz="0.2 ${radius + 0.15} 0" rpy="${180*pi/180}  -${90*pi/180} 0" />
+    <origin xyz="0.2125 0.31 0" rpy="${180*pi/180}  -${90*pi/180} 0" />
   </xacro:T200_macro>
   <!-- Front Right Horizontal Thruster -->
   <xacro:T200_macro thruster_id="7">
-    <origin xyz="0.2 -${radius + 0.15} 0" rpy="0 ${90*pi/180} 0" />
+    <origin xyz="0.2125 -0.31 0" rpy="0 ${90*pi/180} 0" />
   </xacro:T200_macro>
   <xacro:light_macro light_id="0">
-    <origin xyz="0.405 0 0" rpy="0 0 0" />
+    <origin xyz="0.1 0 0" rpy="0 0 0" />
   </xacro:light_macro>
   <!-- Sensors -->
   <!-- Forward Camera -->
   <xacro:camera_macro camera_id="0">
-    <origin xyz="0.305 0 0" rpy="0 0 0" />
+    <origin xyz="0.335 0 0" rpy="0 0 0" />
   </xacro:camera_macro>
   <!-- Downward Camera -->
@@ -91,5 +91,5 @@
   <!-- 360 Top Sonar -->
   <xacro:ping360_macro sonar_id="1">
-    <origin xyz="0 0 ${radius + 0.02}" rpy="0 0 0" />
+    <origin xyz="0 0 ${radius + 0.02 - 0.1}" rpy="0 0 0" />
   </xacro:ping360_macro>
   <!-- IMU -->

Commit message: Add dual camera and new model

File: pontus_description/models/pontus/components/lights.xacro (robot description, xacro)
@@ -19,5 +19,5 @@
             <pose>0 0 0 0 1.57 3.14</pose>
             <attenuation>
-                <range>4</range>
+                <range>10</range>
                 <constant>1</constant>
                 <linear>0.5</linear>

File: pontus_description/models/pontus/components/sensors.xacro (robot description, xacro)
@@ -14,5 +14,5 @@
       <sensor name="camera_${camera_id}" type="camera">
         <camera>
-          <horizontal_fov>1.20428</horizontal_fov>
+          <horizontal_fov>1.3962634</horizontal_fov>
           <image>
             <width>640</width>

File: pontus_description/models/pontus/pontus.xacro (robot description, xacro)
@@ -78,5 +78,8 @@
   <!-- Sensors -->
   <!-- Forward Camera -->
-  <xacro:camera_macro camera_id="0">
+  <xacro:camera_macro camera_id="2">
+    <origin xyz="0.305 0.08 0" rpy="0 0 0" />
+  </xacro:camera_macro>
+    <xacro:camera_macro camera_id="3">
     <origin xyz="0.305 0 0" rpy="0 0 0" />
   </xacro:camera_macro>
