Commit message: Add Sonar, IMU, and camera. Also adds a new testing world and adds all world files to the path

File: pontus_description/models/pontus/components/sensors.xacro (robot description, xacro)
@@ -1,21 +1,128 @@
 <?xml version="1.0"?>
 <robot xmlns:xacro="http://www.ros.org/wiki/xacro">
-  <!-- Pose 3D sensor. -->
-  <xacro:default_pose_3d namespace="${namespace}" parent_link="${namespace}/base_link" />
-  <!-- Forward-looking sonar sensor -->
-  <xacro:forward_multibeam_p900 namespace="${namespace}" topic="${namespace}/sonar_forward" parent_link="${namespace}/base_link">
-  <origin xyz="0 1.35 0" rpy="0 0 ${90*d2r}"/>
-  </xacro:forward_multibeam_p900>
+  <xacro:property name="P900_mesh" value="file://$(find pontus_description)/models/pontus/meshes/p900.dae"/>
+  <!-- Camera  -->
+  <xacro:macro name="camera_macro" params="camera_id *origin">
+    <link name="camera_${camera_id}"/>
+    <joint name="camera_joint_${camera_id}" type="fixed">
+      <xacro:insert_block name="origin"/>
+      <parent link="base_link"/>
+      <child link="camera_${camera_id}"/>
+      <axis xyz="1 0 0"/>
+    </joint>
+    <gazebo reference="camera_${camera_id}">
+      <sensor name="camera_${camera_id}" type="camera">
+        <camera>
+          <horizontal_fov>1.047</horizontal_fov>
+          <image>
+            <width>320</width>
+            <height>240</height>
+          </image>
+          <clip>
+            <near>0.1</near>
+            <far>100</far>
+          </clip>
+        </camera>
+        <always_on>1</always_on>
+        <update_rate>30</update_rate>
+        <visualize>true</visualize>
+        <topic>pontus/camera_${camera_id}</topic>
+      </sensor>
+    </gazebo>
+  </xacro:macro>
+  <!-- P900 Sonar  -->
+  <xacro:macro name="p900_macro" params="sonar_id *origin">
+    <link name="sonar_${sonar_id}">
+     <visual>
+        <geometry>
+          <mesh filename="${P900_mesh}"/>
+        </geometry>
+      </visual>
+    </link>
+    <joint name="sonar_joint_${sonar_id}" type="fixed">
+      <xacro:insert_block name="origin"/>
+      <parent link="base_link"/>
+      <child link="sonar_${sonar_id}"/>
+      <axis xyz="1 0 0"/>
+    </joint>
+    <gazebo reference="sonar_${sonar_id}">
+      <sensor name="sonar_${sonar_id}" type="gpu_lidar">
+        <lidar>
+          <scan>
+            <horizontal>
+              <samples>256</samples>
+              <resolution>1</resolution>
+              <min_angle>-0.3927</min_angle>
+              <max_angle>0.3927</max_angle>
+            </horizontal>
+          </scan>
+          <range>
+            <min>1.0</min>
+            <max>100.0</max>
+            <resolution>0.01</resolution>
+          </range>
+          <noise>
+            <type>gaussian</type>
+            <mean>0.0</mean>
+            <stddev>0.027</stddev>
+          </noise>
+        </lidar>
+        <always_on>1</always_on>
+        <update_rate>15</update_rate>
+        <visualize>true</visualize>
+        <topic>pontus/sonar_${sonar_id}</topic>
+        <!-- This tag isn't recognized by SDF but is extremely important for getting the correct TF data for the sonar frame-->
+        <gz_frame_id>sonar_${sonar_id}</gz_frame_id>
+      </sensor>
+    </gazebo>
+  </xacro:macro>
+  <!-- IMU  -->
+  <xacro:macro name="imu_macro" params="imu_id *origin">
+    <link name="imu_${imu_id}"/>
+    <joint name="imu_joint_${imu_id}" type="fixed">
+      <xacro:insert_block name="origin"/>
+      <parent link="base_link"/>
+      <child link="imu_${imu_id}"/>
+      <axis xyz="1 0 0"/>
+    </joint>
+    <gazebo reference="imu_${imu_id}">
+      <sensor name="imu_sensor" type="imu">
+        <pose>0 0 0 0 0 0</pose>
+        <always_on>1</always_on>
+        <visualize>true</visualize>
+        <enable_metrics>true</enable_metrics>
+        <update_rate>100</update_rate>
+      </sensor>
+    </gazebo>
+  </xacro:macro>
   <!-- Pressure  -->
-  <xacro:default_pressure namespace="${namespace}" parent_link="${namespace}/base_link">
-    <origin xyz="0 0 0" rpy="0 0 0"/>
-  </xacro:default_pressure>
-  <!-- IMU  -->
-  <xacro:default_imu namespace="${namespace}" parent_link="${namespace}/base_link">
-    <origin xyz="0 0 0" rpy="0 0 0"/>
-  </xacro:default_imu>
-  <!-- Camera  -->
-  <xacro:default_camera namespace="${namespace}" parent_link="${namespace}/base_link" suffix="_forward">
-    <origin xyz="0 1.35 0" rpy="0 0 ${90*d2r}"/>
-  </xacro:default_camera>
+  <!-- TODO: Find a way to get pressure/depth reading. This will be important for localization
+             Unfortunately the air_pressure sensor doesn't seem like it will actually work -->
+  <xacro:macro name="pressure_macro" params="pressure_id *origin">
+    <link name="pressure_${pressure_id}"/>
+    <joint name="pressure_joint_${pressure_id}" type="fixed">
+      <xacro:insert_block name="origin"/>
+      <parent link="base_link"/>
+      <child link="pressure_${pressure_id}"/>
+      <axis xyz="1 0 0"/>
+    </joint>
+    <gazebo reference="pressure_${pressure_id}">
+      <sensor name="pressure" type="air_pressure">
+        <always_on>1</always_on>
+        <update_rate>30</update_rate>
+        <visualize>true</visualize>
+        <topic>pressure_${pressure_id}</topic>
+        <enable_metrics>true</enable_metrics>
+        <air_pressure>
+          <reference_altitude>0</reference_altitude>
+          <pressure>
+            <noise type="gaussian">
+              <mean>0.2</mean>
+              <stddev>0.1</stddev>
+            </noise>
+          </pressure>
+        </air_pressure>
+      </sensor>
+    </gazebo>
+  </xacro:macro>
 </robot>

File: pontus_description/models/pontus/components/thrusters.xacro (robot description, xacro)
@@ -6,6 +6,6 @@
     <link name="thruster_${thruster_id}">
       <visual>
-	<geometry>
-	  <mesh filename="${T200_body_mesh}"/>
+        <geometry>
+          <mesh filename="${T200_body_mesh}"/>
         </geometry>
         <material name="Black">

File: pontus_description/models/pontus/pontus.xacro (robot description, xacro)
@@ -2,5 +2,8 @@
 <robot name="pontus" xmlns:xacro="http://www.ros.org/wiki/xacro" >
   <xacro:include filename="$(find pontus_description)/models/pontus/components/thrusters.xacro"/>
+  <xacro:include filename="$(find pontus_description)/models/pontus/components/sensors.xacro"/>
   <!--<xacro:property name="mesh_file" value="file://$(find pontus_description)/models/pontus/meshes/pontus_body_mesh.STL"/>-->
+  <xacro:arg name="sim" default="false"/>
+  <xacro:arg name="static" default="false"/>
   <xacro:property name="fluid_density" value="1025"/>
   <xacro:property name="namespace" value="pontus"/>
@@ -69,7 +72,24 @@
     <origin xyz="0.2 ${radius + 0.15} 0" rpy="${180*pi/180}  ${90*pi/180} 0" />
   </xacro:T200_macro>
-  <!-- TODO: Sensors -->
+  <!-- Sensors -->
+  <!-- Forward Camera -->
+  <xacro:camera_macro camera_id="0">
+    <origin xyz="0.305 0 0" rpy="0 0 0" />
+  </xacro:camera_macro>
+  <!-- Forward Sonar -->
+  <xacro:p900_macro sonar_id="0">
+    <origin xyz="0.28 0 -0.15" rpy="0 ${45*pi/180} 0" />
+  </xacro:p900_macro>
+  <!-- IMU -->
+  <xacro:imu_macro imu_id="0">
+    <origin xyz="0 0 0" rpy="0 0 0" />
+  </xacro:imu_macro>
+  <!-- Pressure -->
+  <xacro:pressure_macro pressure_id="0">
+    <origin xyz="0 0 0" rpy="0 0 0" />
+  </xacro:pressure_macro>
+  <!-- Lock Pontus in place for sensor testing -->
   <gazebo>
-    <static>false</static>
+    <static>$(arg static)</static>
   </gazebo>
   <!-- hydrodynamics and control plugins -->
@@ -79,5 +99,5 @@
       filename="gz-sim-hydrodynamics-system"
       name="gz::sim::systems::Hydrodynamics">
-    <link_name> base_link </link_name>
+      <link_name> base_link </link_name>
       <!-- Incorrect Added Mass values causing crashes -->
       <!--<xDotU>-4.876161</xDotU>

Commit message: Debugging localization, not working

File: pontus_description/models/pontus/components/sensors.xacro (robot description, xacro)
@@ -35,9 +35,9 @@
   <xacro:macro name="p900_macro" params="sonar_id *origin">
     <link name="sonar_${sonar_id}">
-     <visual>
+     <!-- <visual>
         <geometry>
           <mesh filename="${P900_mesh}"/>
         </geometry>
-      </visual>
+      </visual> -->
     </link>
     <joint name="sonar_joint_${sonar_id}" type="fixed">

File: pontus_description/models/pontus/components/thrusters.xacro (robot description, xacro)
@@ -5,5 +5,5 @@
   <xacro:macro name="T200_macro" params="thruster_id *origin">
     <link name="thruster_${thruster_id}">
-      <visual>
+      <!-- <visual>
         <origin xyz="0 0 0" rpy="0 ${180*pi/180} 0"/>
         <geometry>
@@ -13,5 +13,5 @@
           <color rgba="0.0 0.0 0.0 1.0"/>
         </material>
-      </visual>
+      </visual> -->
     </link>
     <joint name="thruster_joint_${thruster_id}" type="fixed">
@@ -28,5 +28,5 @@
                  iyy="0.001" iyz="0.0" izz="0.001" />
       </inertial>
-      <visual>
+      <!-- <visual>
         <origin xyz="0 0 0" rpy="0 ${180*pi/180} 0"/>
         <geometry>
@@ -36,5 +36,5 @@
           <color rgba="0.26 0.46 0.68 1.0"/>
         </material>
-      </visual>
+      </visual> -->
     </link>
     <joint name="prop_joint_${thruster_id}" type="continuous">

File: pontus_description/models/pontus/pontus.xacro (robot description, xacro)
@@ -23,5 +23,5 @@
       />
     </inertial>
-    <visual>
+    <!-- <visual>
       <origin xyz="0 0 0" rpy="0 ${-90*pi/180} 0"/>
       <geometry>
@@ -31,5 +31,5 @@
         <color rgba="0.9 0.9 0.9 0.4"/>
       </material>
-    </visual>
+    </visual> -->
     <collision>
       <origin xyz="0 0 0" rpy="0 ${-90*pi/180} 0"/>
@@ -103,4 +103,5 @@
   <!-- hydrodynamics and control plugins -->
   <gazebo>
+    <cast_shadows>false</cast_shadows>
     <!-- TODO: get actual numbers for this -->
     <plugin

Commit message: Changes

File: pontus_description/models/pontus/components/sensors.xacro (robot description, xacro)
@@ -14,8 +14,8 @@
       <sensor name="camera_${camera_id}" type="camera">
         <camera>
-          <horizontal_fov>1.047</horizontal_fov>
+          <horizontal_fov>1.20427718</horizontal_fov>
           <image>
             <width>320</width>
-            <height>240</height>
+            <height>255</height>
           </image>
           <clip>

File: pontus_description/models/pontus/pontus.xacro (robot description, xacro)
@@ -81,8 +81,4 @@
     <origin xyz="-.28 .0375 -.15" rpy="0 1.57 0" />
   </xacro:camera_macro>
-  <!-- Bottom Camera 2 -->
-  <xacro:camera_macro camera_id="2">
-    <origin xyz="-.28 -.0375 -.15" rpy="0 1.57 0" />
-  </xacro:camera_macro>
   <!-- Forward Sonar -->
   <xacro:p900_macro sonar_id="0">

Commit message: New Autonomy Layout

File: pontus_description/models/pontus/components/sensors.xacro (robot description, xacro)
@@ -31,9 +31,10 @@
     </gazebo>
   </xacro:macro>
-  <!-- P900 Sonar  -->
-  <xacro:macro name="p900_macro" params="sonar_id *origin">
+  <!-- Sonoptix Echo Sonar  -->
+  <xacro:macro name="sonoptix_macro" params="sonar_id *origin">
     <link name="sonar_${sonar_id}">
      <visual>
         <geometry>
+          <!-- TODO: get the right mesh -->
           <mesh filename="${P900_mesh}"/>
         </geometry>
@@ -53,11 +54,59 @@
               <samples>256</samples>
               <resolution>1</resolution>
-              <min_angle>-0.3927</min_angle>
-              <max_angle>0.3927</max_angle>
+              <min_angle>-1.0472</min_angle>
+              <max_angle>1.0472</max_angle>
             </horizontal>
           </scan>
           <range>
-            <min>1.0</min>
-            <max>100.0</max>
+            <min>0.2</min>
+            <max>30.0</max>
+            <resolution>0.008</resolution>
+          </range>
+          <noise>
+            <type>gaussian</type>
+            <mean>0.0</mean>
+            <stddev>0.027</stddev>
+          </noise>
+        </lidar>
+        <always_on>1</always_on>
+        <update_rate>25</update_rate>
+        <visualize>true</visualize>
+        <topic>pontus/sonar_${sonar_id}</topic>
+        <!-- This tag isn't recognized by SDF but is extremely important for getting the correct TF data for the sonar frame-->
+        <gz_frame_id>sonar_${sonar_id}</gz_frame_id>
+      </sensor>
+    </gazebo>
+  </xacro:macro>
+  <!-- Ping360 Sonar  -->
+  <xacro:macro name="ping360_macro" params="sonar_id *origin">
+    <link name="sonar_${sonar_id}">
+     <visual>
+      <origin xyz="0 0 0" rpy="0 ${-90*pi/180} 0"/>
+        <geometry>
+          <!-- TODO: get the right mesh -->
+          <mesh filename="${P900_mesh}" scale="0.3 0.3 0.3"/>
+        </geometry>
+      </visual>
+    </link>
+    <joint name="sonar_joint_${sonar_id}" type="fixed">
+      <xacro:insert_block name="origin"/>
+      <parent link="base_link"/>
+      <child link="sonar_${sonar_id}"/>
+      <axis xyz="1 0 0"/>
+    </joint>
+    <gazebo reference="sonar_${sonar_id}">
+      <sensor name="sonar_${sonar_id}" type="gpu_lidar">
+        <lidar>
+          <scan>
+            <horizontal>
+              <samples>180</samples>
+              <resolution>1</resolution>
+              <min_angle>-3.14159</min_angle>
+              <max_angle>3.14159</max_angle>
+            </horizontal>
+          </scan>
+          <range>
+            <min>0.75</min>
+            <max>50.0</max>
             <resolution>0.01</resolution>
           </range>
@@ -69,5 +118,6 @@
         </lidar>
         <always_on>1</always_on>
-        <update_rate>15</update_rate>
+        <!-- The ping360 sweeps a single beam, we would have to simulate it with physically rotating the lidar. This is easier for now-->
+        <update_rate>1</update_rate>
         <visualize>true</visualize>
         <topic>pontus/sonar_${sonar_id}</topic>

File: pontus_description/models/pontus/pontus.xacro (robot description, xacro)
@@ -78,7 +78,11 @@
   </xacro:camera_macro>
   <!-- Forward Sonar -->
-  <xacro:p900_macro sonar_id="0">
+  <xacro:sonoptix_macro sonar_id="0">
     <origin xyz="0.28 0 -0.15" rpy="0 ${45*pi/180} 0" />
-  </xacro:p900_macro>
+  </xacro:sonoptix_macro>
+  <!-- 360 Top Sonar -->
+  <xacro:ping360_macro sonar_id="1">
+    <origin xyz="0 0 ${radius + 0.02}" rpy="0 0 0" />
+  </xacro:ping360_macro>
   <!-- IMU -->
   <xacro:imu_macro imu_id="0">

Commit message: New nuc changes

File: pontus_description/models/pontus/components/sensors.xacro (robot description, xacro)
@@ -30,4 +30,14 @@
       </sensor>
     </gazebo>
+  </xacro:macro>
+  <!-- DVL  -->
+  <xacro:macro name="dvl_macro" params="dvl_id *origin">
+    <link name="dvl_a50_link"/>
+    <joint name="dvl_joint_${dvl_id}" type="fixed">
+      <xacro:insert_block name="origin"/>
+      <parent link="base_link"/>
+      <child link="dvl_a50_link"/>
+      <axis xyz="1 0 0"/>
+    </joint>
   </xacro:macro>
   <!-- P900 Sonar  -->

File: pontus_description/models/pontus/pontus.xacro (robot description, xacro)
@@ -81,4 +81,8 @@
     <origin xyz="0.28 0 -0.15" rpy="0 ${45*pi/180} 0" />
   </xacro:p900_macro>
+  <!-- DVL -->
+  <xacro:dvl_macro dvl_id="0">
+    <origin xyz="0 0 0" rpy="0 0 0" />
+  </xacro:dvl_macro>
   <!-- IMU -->
   <xacro:imu_macro imu_id="0">

Commit message: Add Pontus model to sim and argument for sim PID values

File: pontus_description/models/pontus/components/sensors.xacro (robot description, xacro)
@@ -41,5 +41,5 @@
     </joint>
   </xacro:macro>
-  <!-- P900 Sonar  -->
+  <!-- Sonoptix Echo  -->
   <xacro:macro name="sonoptix_macro" params="sonar_id *origin">
     <link name="sonar_${sonar_id}">

File: pontus_description/models/pontus/pontus.xacro (robot description, xacro)
@@ -87,5 +87,5 @@
   <!-- Forward Sonar -->
   <xacro:sonoptix_macro sonar_id="0">
-    <origin xyz="0.28 0 -0.15" rpy="0 ${25*pi/180} 0" />
+    <origin xyz="0.28 0 -0.15" rpy="${pi} ${25*pi/180} 0" />
   </xacro:sonoptix_macro>
   <!-- 360 Top Sonar -->

File: pontus_description/models/pontus/pontus_real.xacro (robot description, xacro)
@@ -9,5 +9,5 @@
   <xacro:property name="fluid_density" value="1025"/>
   <xacro:property name="namespace" value="pontus"/>
-  <xacro:property name="mass" value="155"/>
+  <xacro:property name="mass" value="156"/>
   <xacro:property name="length" value="0.78"/>
   <xacro:property name="radius" value="0.25"/>
@@ -21,6 +21,6 @@
       <!-- TODO: insert actual calculations instead of precalculated value -->
       <inertia
-        ixx="55" ixy="0" ixz="0"
-        iyy="0.585" iyz="0" izz="55"
+        ixx="156" ixy="0" ixz="0"
+        iyy="0.585" iyz="0" izz="156"
       />
     </inertial>

Commit message: Fixes camera optical tfs, cluster coord close to working

File: pontus_description/models/pontus/components/sensors.xacro (robot description, xacro)
@@ -11,4 +11,10 @@
       <axis xyz="1 0 0"/>
     </joint>
+    <joint name="camera_${camera_id}_optical_frame_joint" type="fixed">
+      <origin xyz="0 0 0" rpy="${-pi/2} 0.0 ${-pi/2}" />
+      <parent link="camera_${camera_id}" />
+      <child link="camera_${camera_id}_optical_frame"/>
+    </joint>
+    <link name="camera_${camera_id}_optical_frame"/>
     <gazebo reference="camera_${camera_id}">
       <sensor name="camera_${camera_id}" type="camera">
@@ -23,4 +29,6 @@
             <far>100</far>
           </clip>
+          <optical_frame_id>camera_${camera_id}_optical_frame</optical_frame_id>
+          <camera_info_topic>pontus/camera_${camera_id}/camera_info</camera_info_topic>
         </camera>
         <always_on>1</always_on>

File: pontus_description/models/pontus/pontus.xacro (robot description, xacro)
@@ -95,5 +95,5 @@
   <!-- Forward Camera -->
   <xacro:camera_macro camera_id="front">
-    <origin xyz="0.305 0 0" rpy="0 0 0" />
+    <origin xyz="0.305 0.075 0" rpy="0 0 0" />
   </xacro:camera_macro>
   <xacro:camera_macro camera_id="3">
