Commit message: DVL command client, dvl drift correction node

File: pontus_description/models/pontus/components/sensors.xacro (robot description, xacro)
@@ -181,9 +181,14 @@
     <gazebo reference="imu_${imu_id}">
       <sensor name="imu_sensor" type="imu">
+        <imu>
+          <orientation_reference_frame>
+            <localization>ENU</localization>
+            <custom_rpy>0 0 0</custom_rpy>
+          </orientation_reference_frame>
+        </imu>
         <pose>0 0 0 0 0 0</pose>
         <always_on>1</always_on>
         <visualize>true</visualize>
         <topic>pontus/imu_${imu_id}</topic>
-        <enable_metrics>true</enable_metrics>
         <update_rate>100</update_rate>
         <!-- This tag isn't recognized by SDF but is extremely important for getting the correct TF data for the IMU frame-->

File: pontus_description/models/pontus/pontus.xacro (robot description, xacro)
@@ -142,5 +142,5 @@
   <!-- IMU -->
   <xacro:imu_macro imu_id="0">
-    <origin xyz="0 0 0" rpy="1.571 0 -1.571" />
+    <origin xyz="0 0 0" rpy="0 0 0" />
   </xacro:imu_macro>
   <!-- Pressure -->
