Commit message: Remove new pontus model

File: pontus_description/models/pontus/pontus_real.xacro (robot description, xacro)
@@ -4,12 +4,12 @@
   <xacro:include filename="$(find pontus_description)/models/pontus/components/sensors.xacro"/>
   <xacro:include filename="$(find pontus_description)/models/pontus/components/lights.xacro"/>
-  <!--<xacro:property name="mesh_file" value="file://$(find pontus_description)/models/pontus/meshes/pontus_body_mesh.STL"/>-->
+  <xacro:property name="mesh_file" value="file://$(find pontus_description)/models/pontus/meshes/tech_triton.STL"/>
   <xacro:arg name="sim" default="false"/>
   <xacro:arg name="static" default="false"/>
   <xacro:property name="fluid_density" value="1025"/>
   <xacro:property name="namespace" value="pontus"/>
-  <xacro:property name="mass" value="50"/>
-  <xacro:property name="length" value="0.61"/>
-  <xacro:property name="radius" value="0.1"/>
+  <xacro:property name="mass" value="155"/>
+  <xacro:property name="length" value="0.78"/>
+  <xacro:property name="radius" value="0.25"/>
   <xacro:property name="volume" value="${pi*length*(radius)**2}"/>
   <!-- Create pontus -->
@@ -17,5 +17,6 @@
     <inertial>
       <!-- This is calculated for slightly positive buoyancy -->
-      <mass value="${(volume * fluid_density) - 1.0}"/>
+      <!-- <mass value="${(volume * fluid_density) - 1.0}"/> -->
+      <mass value="${mass}"/>
       <!-- TODO: insert actual calculations instead of precalculated value -->
       <inertia
@@ -25,10 +26,10 @@
     </inertial>
     <visual>
-      <origin xyz="0 0 0" rpy="0 ${-90*pi/180} 0"/>
+      <origin xyz="-0.346957 -0.271635 -0.1620155" rpy="1.57 0 1.57"/>
       <geometry>
-        <cylinder length="${length}" radius="${radius}"/>
+        <mesh filename="${mesh_file}" scale="1 1 1"/>
       </geometry>
       <material name="acrylic">
-        <color rgba="0.9 0.9 0.9 0.4"/>
+        <color rgba="0.5 0.5 0.5 0.8"/>
       </material>
     </visual>
@@ -43,33 +44,33 @@
   <!-- Back Left Vertical Thruster -->
   <xacro:T200_macro thruster_id="0">
-    <origin xyz="-0.075 -${radius + 0.07} 0" rpy="0 0 0" />
+    <origin xyz="-0.0775 -0.2 0" rpy="0 0 0" />
   </xacro:T200_macro>
   <!-- Back Right Vertical Thruster -->
   <xacro:T200_macro thruster_id="1">
-    <origin xyz="-0.075 ${radius + 0.07} 0" rpy="0 0 ${180*pi/180}" />
+    <origin xyz="-0.0775 0.2 0" rpy="0 0 ${180*pi/180}" />
   </xacro:T200_macro>
   <!-- Front Left Vertical Thruster -->
   <xacro:T200_macro thruster_id="2">
-    <origin xyz="0.075 -${radius + 0.07} 0" rpy="0 0 0" />
+    <origin xyz="0.0775 -0.2 0" rpy="0 0 0" />
   </xacro:T200_macro>
   <!-- Front Right Vertical Thruster -->
   <xacro:T200_macro thruster_id="3">
-    <origin xyz="0.075 ${radius + 0.07} 0" rpy="0 0 ${180*pi/180}" />
+    <origin xyz="0.0775 0.2 0" rpy="0 0 ${180*pi/180}" />
   </xacro:T200_macro>
   <!-- Back Left Horizontal Thruster -->
   <xacro:T200_macro thruster_id="4">
-    <origin xyz="-0.2 ${radius + 0.15} 0" rpy="${180*pi/180}  -${90*pi/180} 0" />
+    <origin xyz="-0.2295 0.31 0" rpy="${180*pi/180}  -${90*pi/180} 0" />
   </xacro:T200_macro>
   <!-- Back Right Horizontal Thruster -->
   <xacro:T200_macro thruster_id="5">
-    <origin xyz="-0.2 -${radius + 0.15} 0" rpy="0 ${90*pi/180} 0" />
+    <origin xyz="-0.2295 -0.31 0" rpy="0 ${90*pi/180} 0" />
   </xacro:T200_macro>
   <!-- Front Left Horizontal Thruster -->
   <xacro:T200_macro thruster_id="6">
-    <origin xyz="0.2 ${radius + 0.15} 0" rpy="${180*pi/180}  -${90*pi/180} 0" />
+    <origin xyz="0.2125 0.31 0" rpy="${180*pi/180}  -${90*pi/180} 0" />
   </xacro:T200_macro>
   <!-- Front Right Horizontal Thruster -->
   <xacro:T200_macro thruster_id="7">
-    <origin xyz="0.2 -${radius + 0.15} 0" rpy="0 ${90*pi/180} 0" />
+    <origin xyz="0.2125 -0.31 0" rpy="0 ${90*pi/180} 0" />
   </xacro:T200_macro>
   <xacro:light_macro light_id="0">
@@ -79,5 +80,5 @@
   <!-- Forward Camera -->
   <xacro:camera_macro camera_id="0">
-    <origin xyz="0.305 0 0" rpy="0 0 0" />
+    <origin xyz="0.335 0 0" rpy="0 0 0" />
   </xacro:camera_macro>
   <!-- Downward Camera -->
@@ -91,5 +92,5 @@
   <!-- 360 Top Sonar -->
   <xacro:ping360_macro sonar_id="1">
-    <origin xyz="0 0 ${radius + 0.02}" rpy="0 0 0" />
+    <origin xyz="0 0 ${radius + 0.02 - 0.1}" rpy="0 0 0" />
   </xacro:ping360_macro>
   <!-- IMU -->

Commit message: Add sonoptix driver paramaters and laserscan message publisher

File: pontus_description/models/pontus/pontus_real.xacro (robot description, xacro)
@@ -94,4 +94,8 @@
     <origin xyz="0 0 ${radius + 0.02 - 0.1}" rpy="0 0 0" />
   </xacro:ping360_macro>
+  <!-- DVL -->
+  <xacro:dvl_macro dvl_id="0">
+    <origin xyz="0 0 0" rpy="0 0 0" />
+  </xacro:dvl_macro>
   <!-- IMU -->
   <xacro:imu_macro imu_id="0">
