Commit message: Added lane markers to make the bottom of the pool a grid and attempted to add camera (not working)

File: pontus_description/models/pontus/pontus.xacro (robot description, xacro)
@@ -77,4 +77,8 @@
     <origin xyz="0.305 0 0" rpy="0 0 0" />
   </xacro:camera_macro>
+  <!-- Bottom Camera -->
+  <xacro:camera_macro camera_id="1">
+    <origin xyz="-.28 0 -.15" rpy="0 0 0" />
+  </xacro:camera_macro>
   <!-- Forward Sonar -->
   <xacro:p900_macro sonar_id="0">

Commit message: Fixed the camera by adding into the bridge.yml file in the pontus_sim package. This allows for the ros_gz_bridge to match the gazebo topic to the ros topic

File: pontus_description/models/pontus/pontus.xacro (robot description, xacro)
@@ -79,5 +79,5 @@
   <!-- Bottom Camera -->
   <xacro:camera_macro camera_id="1">
-    <origin xyz="-.28 0 -.15" rpy="0 0 0" />
+    <origin xyz="-.28 0 -.15" rpy="0 1.57 0" />
   </xacro:camera_macro>
   <!-- Forward Sonar -->

Commit message: Added extra camera to bottom of sub

File: pontus_description/models/pontus/pontus.xacro (robot description, xacro)
@@ -77,7 +77,11 @@
     <origin xyz="0.305 0 0" rpy="0 0 0" />
   </xacro:camera_macro>
-  <!-- Bottom Camera -->
+  <!-- Bottom Camera 1 -->
   <xacro:camera_macro camera_id="1">
-    <origin xyz="-.28 0 -.15" rpy="0 1.57 0" />
+    <origin xyz="-.28 .0375 -.15" rpy="0 1.57 0" />
+  </xacro:camera_macro>
+  <!-- Bottom Camera 2 -->
+  <xacro:camera_macro camera_id="2">
+    <origin xyz="-.28 -.0375 -.15" rpy="0 1.57 0" />
   </xacro:camera_macro>
   <!-- Forward Sonar -->

Commit message: Some particle filter

File: pontus_description/models/pontus/pontus.xacro (robot description, xacro)
@@ -23,5 +23,5 @@
       />
     </inertial>
-    <!-- <visual>
+    <visual>
       <origin xyz="0 0 0" rpy="0 ${-90*pi/180} 0"/>
       <geometry>
@@ -31,5 +31,5 @@
         <color rgba="0.9 0.9 0.9 0.4"/>
       </material>
-    </visual> -->
+    </visual>
     <collision>
       <origin xyz="0 0 0" rpy="0 ${-90*pi/180} 0"/>

Commit message: Swap horizontal thruster locations in sim to match what it was supposed to be

File: pontus_description/models/pontus/pontus.xacro (robot description, xacro)
@@ -58,17 +58,17 @@
   <!-- Back Left Horizontal Thruster -->
   <xacro:T200_macro thruster_id="4">
-    <origin xyz="-0.2 -${radius + 0.15} 0" rpy="0 ${90*pi/180} 0" />
+    <origin xyz="-0.2 ${radius + 0.15} 0" rpy="${180*pi/180}  -${90*pi/180} 0" />
   </xacro:T200_macro>
   <!-- Back Right Horizontal Thruster -->
   <xacro:T200_macro thruster_id="5">
-    <origin xyz="-0.2 ${radius + 0.15} 0" rpy="${180*pi/180}  -${90*pi/180} 0" />
+    <origin xyz="-0.2 -${radius + 0.15} 0" rpy="0 ${90*pi/180} 0" />
   </xacro:T200_macro>
   <!-- Front Left Horizontal Thruster -->
   <xacro:T200_macro thruster_id="6">
-    <origin xyz="0.2 -${radius + 0.15} 0" rpy="0 ${90*pi/180} 0" />
+    <origin xyz="0.2 ${radius + 0.15} 0" rpy="${180*pi/180}  -${90*pi/180} 0" />
   </xacro:T200_macro>
   <!-- Front Right Horizontal Thruster -->
   <xacro:T200_macro thruster_id="7">
-    <origin xyz="0.2 ${radius + 0.15} 0" rpy="${180*pi/180}  -${90*pi/180} 0" />
+    <origin xyz="0.2 -${radius + 0.15} 0" rpy="0 ${90*pi/180} 0" />
   </xacro:T200_macro>
   <!-- Sensors -->

Commit message: Line detection works

File: pontus_description/models/pontus/pontus.xacro (robot description, xacro)
@@ -79,5 +79,5 @@
   <!-- Bottom Camera 1 -->
   <xacro:camera_macro camera_id="1">
-    <origin xyz="-.28 .0375 -.15" rpy="0 1.57 0" />
+    <origin xyz="0 0 -.15" rpy="0 1.57 0" />
   </xacro:camera_macro>
   <!-- Forward Sonar -->

Commit message: Add downward facing camera

File: pontus_description/models/pontus/pontus.xacro (robot description, xacro)
@@ -77,4 +77,8 @@
     <origin xyz="0.305 0 0" rpy="0 0 0" />
   </xacro:camera_macro>
+  <!-- Downward Camera -->
+  <xacro:camera_macro camera_id="1">
+    <origin xyz="0 0 -0.1" rpy="0 ${90*pi/180} 0" />
+  </xacro:camera_macro>
   <!-- Forward Sonar -->
   <xacro:sonoptix_macro sonar_id="0">

Commit message: Add subsea lights and turn off outside lighting

File: pontus_description/models/pontus/pontus.xacro (robot description, xacro)
@@ -3,4 +3,5 @@
   <xacro:include filename="$(find pontus_description)/models/pontus/components/thrusters.xacro"/>
   <xacro:include filename="$(find pontus_description)/models/pontus/components/sensors.xacro"/>
+  <xacro:include filename="$(find pontus_description)/models/pontus/components/lights.xacro"/>
   <!--<xacro:property name="mesh_file" value="file://$(find pontus_description)/models/pontus/meshes/pontus_body_mesh.STL"/>-->
   <xacro:arg name="sim" default="false"/>
@@ -72,4 +73,7 @@
     <origin xyz="0.2 -${radius + 0.15} 0" rpy="0 ${90*pi/180} 0" />
   </xacro:T200_macro>
+  <xacro:light_macro light_id="0">
+    <origin xyz="0.405 0 0" rpy="0 0 0" />
+  </xacro:light_macro>
   <!-- Sensors -->
   <!-- Forward Camera -->

Commit message: Decrease sonoptix angle

File: pontus_description/models/pontus/pontus.xacro (robot description, xacro)
@@ -87,5 +87,5 @@
   <!-- Forward Sonar -->
   <xacro:sonoptix_macro sonar_id="0">
-    <origin xyz="0.28 0 -0.15" rpy="0 ${45*pi/180} 0" />
+    <origin xyz="0.28 0 -0.15" rpy="0 ${25*pi/180} 0" />
   </xacro:sonoptix_macro>
   <!-- 360 Top Sonar -->

Commit message: Working gate task

File: pontus_description/models/pontus/pontus.xacro (robot description, xacro)
@@ -87,5 +87,5 @@
   <!-- Forward Sonar -->
   <xacro:sonoptix_macro sonar_id="0">
-    <origin xyz="0.28 0 -0.15" rpy="${pi} ${25*pi/180} 0" />
+    <origin xyz="0.28 0 -0.15" rpy="${pi} ${10*pi/180} 0" />
   </xacro:sonoptix_macro>
   <!-- 360 Top Sonar -->

File: pontus_description/models/pontus/pontus_real.xacro (robot description, xacro)
@@ -88,5 +88,5 @@
   <!-- Forward Sonar -->
   <xacro:sonoptix_macro sonar_id="0">
-    <origin xyz="0.28 0 -0.15" rpy="0 ${25*pi/180} 0" />
+    <origin xyz="0.28 0 -0.15" rpy="0 ${10*pi/180} 0" />
   </xacro:sonoptix_macro>
   <!-- 360 Top Sonar -->

Commit message: Modify gate logic to turn first, added stereo camera calculations

File: pontus_description/models/pontus/pontus.xacro (robot description, xacro)
@@ -79,8 +79,8 @@
   <!-- Forward Camera -->
   <xacro:camera_macro camera_id="2">
-    <origin xyz="0.305 0.08 0" rpy="0 0 0" />
+    <origin xyz="0.305 0.375 0" rpy="0 0 0" />
   </xacro:camera_macro>
     <xacro:camera_macro camera_id="3">
-    <origin xyz="0.305 0 0" rpy="0 0 0" />
+    <origin xyz="0.305 -0.0375 0" rpy="0 0 0" />
   </xacro:camera_macro>
   <!-- Downward Camera -->

Commit message: Add side camera to sim

File: pontus_description/models/pontus/pontus.xacro (robot description, xacro)
@@ -79,8 +79,15 @@
   <!-- Forward Camera -->
   <xacro:camera_macro camera_id="2">
-    <origin xyz="0.305 0.375 0" rpy="0 0 0" />
+    <origin xyz="0.305 0.0375 0" rpy="0 0 0" />
   </xacro:camera_macro>
     <xacro:camera_macro camera_id="3">
     <origin xyz="0.305 -0.0375 0" rpy="0 0 0" />
+  </xacro:camera_macro>
+  <!-- Side Camera -->
+  <xacro:camera_macro camera_id="4">
+    <origin xyz="0 0.06 0.1" rpy="0 0 ${90*pi/180}" />
+  </xacro:camera_macro>
+  <xacro:camera_macro camera_id="5">
+    <origin xyz="0 -0.06 0.1" rpy="0 0 -${90*pi/180}" />
   </xacro:camera_macro>
   <!-- Downward Camera -->

Commit message: Add disparity map calculation

File: pontus_description/models/pontus/pontus.xacro (robot description, xacro)
@@ -79,8 +79,8 @@
   <!-- Forward Camera -->
   <xacro:camera_macro camera_id="2">
-    <origin xyz="0.305 0.0375 0" rpy="0 0 0" />
+    <origin xyz="0.305 0 0" rpy="0 0 0" />
   </xacro:camera_macro>
     <xacro:camera_macro camera_id="3">
-    <origin xyz="0.305 -0.0375 0" rpy="0 0 0" />
+    <origin xyz="0.305 -0.075 0" rpy="0 0 0" />
   </xacro:camera_macro>
   <!-- Side Camera -->

Commit message: Add xdrive and strafe to sim

File: pontus_description/models/pontus/pontus.xacro (robot description, xacro)
@@ -59,17 +59,17 @@
   <!-- Back Left Horizontal Thruster -->
   <xacro:T200_macro thruster_id="4">
-    <origin xyz="-0.2 ${radius + 0.15} 0" rpy="${180*pi/180}  -${90*pi/180} 0" />
+    <origin xyz="-0.25 ${radius + 0.15} 0" rpy="${180*pi/180}  -${90*pi/180} ${5/4 * pi}" />
   </xacro:T200_macro>
   <!-- Back Right Horizontal Thruster -->
   <xacro:T200_macro thruster_id="5">
-    <origin xyz="-0.2 -${radius + 0.15} 0" rpy="0 ${90*pi/180} 0" />
+    <origin xyz="-0.25 -${radius + 0.15} 0" rpy="0 ${90*pi/180} ${3/4 * pi}" />
   </xacro:T200_macro>
   <!-- Front Left Horizontal Thruster -->
   <xacro:T200_macro thruster_id="6">
-    <origin xyz="0.2 ${radius + 0.15} 0" rpy="${180*pi/180}  -${90*pi/180} 0" />
+    <origin xyz="0.25 ${radius + 0.15} 0" rpy="${180*pi/180}  -${90*pi/180} ${-1/4 * pi}" />
   </xacro:T200_macro>
   <!-- Front Right Horizontal Thruster -->
   <xacro:T200_macro thruster_id="7">
-    <origin xyz="0.2 -${radius + 0.15} 0" rpy="0 ${90*pi/180} 0" />
+    <origin xyz="0.25 -${radius + 0.15} 0" rpy="0 ${90*pi/180} ${1/4 * pi}" />
   </xacro:T200_macro>
   <xacro:light_macro light_id="0">

Commit message: Jetson changes

File: pontus_description/models/pontus/pontus.xacro (robot description, xacro)
@@ -105,9 +105,9 @@
   <!-- DVL -->
   <xacro:dvl_macro dvl_id="0">
-    <origin xyz="0 0 0" rpy="0 0 0" />
+    <origin xyz="0 0 0" rpy="3.141 0 0" />
   </xacro:dvl_macro>
   <!-- IMU -->
   <xacro:imu_macro imu_id="0">
-    <origin xyz="0 0 0" rpy="0 0 0" />
+    <origin xyz="0 0 0" rpy="1.571 0 -1.571" />
   </xacro:imu_macro>
   <!-- Pressure -->

Commit message: Update gate autonomy

File: pontus_description/models/pontus/pontus.xacro (robot description, xacro)
@@ -9,5 +9,5 @@
   <xacro:property name="fluid_density" value="1025"/>
   <xacro:property name="namespace" value="pontus"/>
-  <xacro:property name="mass" value="50"/>
+  <xacro:property name="mass" value="34.0194"/>
   <xacro:property name="length" value="0.61"/>
   <xacro:property name="radius" value="0.1"/>
@@ -17,5 +17,5 @@
     <inertial>
       <!-- This is calculated for slightly positive buoyancy -->
-      <mass value="${(volume * fluid_density) - 1.0}"/>
+      <mass value="${(volume * fluid_density) - 5.0}"/>
       <!-- TODO: insert actual calculations instead of precalculated value -->
       <inertia
@@ -152,6 +152,6 @@
         <kPabsP>-0.1916</kPabsP>
         <mQabsQ>-63</mQabsQ>
-        <nRabsR>-63</nRabsR>
-            </plugin>
+        <nRabsR>-500</nRabsR>
+      </plugin>
     <!-- Publishes perfect odometry data for testing controllers -->
     <plugin

Commit message: Sub changes 4/4

File: pontus_description/models/pontus/pontus.xacro (robot description, xacro)
@@ -105,5 +105,5 @@
   <!-- DVL -->
   <xacro:dvl_macro dvl_id="0">
-    <origin xyz="0 0 0" rpy="3.141 0 0" />
+    <origin xyz="-0.19685 0 0" rpy="3.141 0 0" />
   </xacro:dvl_macro>
   <!-- IMU -->

Commit message: Fix bugs

File: pontus_description/models/pontus/pontus.xacro (robot description, xacro)
@@ -153,4 +153,5 @@
         <mQabsQ>-63</mQabsQ>
         <nRabsR>-500</nRabsR>
+        <!-- <default_current>-0.05 -0.7 0.0</default_current> -->
       </plugin>
     <!-- Publishes perfect odometry data for testing controllers -->

File: pontus_description/models/pontus/pontus_real.xacro (robot description, xacro)
@@ -9,7 +9,7 @@
   <xacro:property name="fluid_density" value="1025"/>
   <xacro:property name="namespace" value="pontus"/>
-  <xacro:property name="mass" value="156"/>
-  <xacro:property name="length" value="0.78"/>
-  <xacro:property name="radius" value="0.25"/>
+  <xacro:property name="mass" value="34.0194"/>
+  <xacro:property name="length" value="0.61"/>
+  <xacro:property name="radius" value="0.1"/>
   <xacro:property name="volume" value="${pi*length*(radius)**2}"/>
   <!-- Create pontus -->
@@ -17,10 +17,9 @@
     <inertial>
       <!-- This is calculated for slightly positive buoyancy -->
-      <!-- <mass value="${(volume * fluid_density) - 1.0}"/> -->
-      <mass value="${mass}"/>
+      <mass value="${(volume * fluid_density) - 5.0}"/>
       <!-- TODO: insert actual calculations instead of precalculated value -->
       <inertia
-        ixx="156" ixy="0" ixz="0"
-        iyy="0.585" iyz="0" izz="156"
+        ixx="55" ixy="0" ixz="0"
+        iyy="0.585" iyz="0" izz="55"
       />
     </inertial>
@@ -44,33 +43,33 @@
   <!-- Back Left Vertical Thruster -->
   <xacro:T200_macro thruster_id="0">
-    <origin xyz="-0.0775 -0.2 0" rpy="0 0 0" />
+    <origin xyz="-0.075 -${radius + 0.07} 0" rpy="0 0 0" />
   </xacro:T200_macro>
   <!-- Back Right Vertical Thruster -->
   <xacro:T200_macro thruster_id="1">
-    <origin xyz="-0.0775 0.2 0" rpy="0 0 ${180*pi/180}" />
+    <origin xyz="-0.075 ${radius + 0.07} 0" rpy="0 0 ${180*pi/180}" />
   </xacro:T200_macro>
   <!-- Front Left Vertical Thruster -->
   <xacro:T200_macro thruster_id="2">
-    <origin xyz="0.0775 -0.2 0" rpy="0 0 0" />
+    <origin xyz="0.075 -${radius + 0.07} 0" rpy="0 0 0" />
   </xacro:T200_macro>
   <!-- Front Right Vertical Thruster -->
   <xacro:T200_macro thruster_id="3">
-    <origin xyz="0.0775 0.2 0" rpy="0 0 ${180*pi/180}" />
+    <origin xyz="0.075 ${radius + 0.07} 0" rpy="0 0 ${180*pi/180}" />
   </xacro:T200_macro>
   <!-- Back Left Horizontal Thruster -->
   <xacro:T200_macro thruster_id="4">
-    <origin xyz="-0.2295 0.31 0" rpy="${180*pi/180}  -${90*pi/180} 0" />
+    <origin xyz="-0.25 ${radius + 0.15} 0" rpy="${180*pi/180}  -${90*pi/180} ${5/4 * pi}" />
   </xacro:T200_macro>
   <!-- Back Right Horizontal Thruster -->
   <xacro:T200_macro thruster_id="5">
-    <origin xyz="-0.2295 -0.31 0" rpy="0 ${90*pi/180} 0" />
+    <origin xyz="-0.25 -${radius + 0.15} 0" rpy="0 ${90*pi/180} ${3/4 * pi}" />
   </xacro:T200_macro>
   <!-- Front Left Horizontal Thruster -->
   <xacro:T200_macro thruster_id="6">
-    <origin xyz="0.2125 0.31 0" rpy="${180*pi/180}  -${90*pi/180} 0" />
+    <origin xyz="0.25 ${radius + 0.15} 0" rpy="${180*pi/180}  -${90*pi/180} ${-1/4 * pi}" />
   </xacro:T200_macro>
   <!-- Front Right Horizontal Thruster -->
   <xacro:T200_macro thruster_id="7">
-    <origin xyz="0.2125 -0.31 0" rpy="0 ${90*pi/180} 0" />
+    <origin xyz="0.25 -${radius + 0.15} 0" rpy="0 ${90*pi/180} ${1/4 * pi}" />
   </xacro:T200_macro>
   <xacro:light_macro light_id="0">
@@ -79,6 +78,16 @@
   <!-- Sensors -->
   <!-- Forward Camera -->
-  <xacro:camera_macro camera_id="0">
-    <origin xyz="0.335 0 0" rpy="0 0 0" />
+  <xacro:camera_macro camera_id="2">
+    <origin xyz="0.35 0 0" rpy="0 0 0" />
+  </xacro:camera_macro>
+    <xacro:camera_macro camera_id="3">
+    <origin xyz="0.35 -0.075 0" rpy="0 0 0" />
+  </xacro:camera_macro>
+  <!-- Side Camera -->
+  <xacro:camera_macro camera_id="4">
+    <origin xyz="0 0.06 0.1" rpy="0 0 ${90*pi/180}" />
+  </xacro:camera_macro>
+  <xacro:camera_macro camera_id="5">
+    <origin xyz="0 -0.06 0.1" rpy="0 0 -${90*pi/180}" />
   </xacro:camera_macro>
   <!-- Downward Camera -->
@@ -88,17 +97,17 @@
   <!-- Forward Sonar -->
   <xacro:sonoptix_macro sonar_id="0">
-    <origin xyz="0.28 0 -0.15" rpy="0 ${10*pi/180} 0" />
+    <origin xyz="0.28 0 -0.15" rpy="${pi} ${10*pi/180} 0" />
   </xacro:sonoptix_macro>
   <!-- 360 Top Sonar -->
   <xacro:ping360_macro sonar_id="1">
-    <origin xyz="0 0 ${radius + 0.02 - 0.1}" rpy="0 0 0" />
+    <origin xyz="0 0 ${radius + 0.02}" rpy="0 0 0" />
   </xacro:ping360_macro>
   <!-- DVL -->
   <xacro:dvl_macro dvl_id="0">
-    <origin xyz="0 0 0" rpy="0 0 0" />
+    <origin xyz="0 0 0" rpy="3.141 0 0" />
   </xacro:dvl_macro>
   <!-- IMU -->
   <xacro:imu_macro imu_id="0">
-    <origin xyz="0 0 0" rpy="0 0 0" />
+    <origin xyz="0 0 0" rpy="1.571 0 -1.571" />
   </xacro:imu_macro>
   <!-- Pressure -->
@@ -132,24 +141,22 @@
         <nDotR>0</nDotR>
         <!-- Linear Drag -->
-        <xU>-10</xU>
-        <yV>-10</yV>
-        <zW>-10</zW>
+        <xU>-5</xU>
+        <yV>-5</yV>
+        <zW>-5</zW>
         <kP>-10</kP>
-        <mQ>-10</mQ>
-        <nR>-10</nR>
-        <!-- Quadratic Drag -->
+        <mQ>-5</mQ>
+        <nR>-5</nR>
         <xUabsU>-6.2282</xUabsU>
-        <yVabsV>-601.27</yVabsV>
-        <zWabsW>-601.27</zWabsW>
+        <yVabsV>-60</yVabsV>
+        <zWabsW>-60</zWabsW>
         <kPabsP>-0.1916</kPabsP>
-        <mQabsQ>-632.698957</mQabsQ>
-        <nRabsR>-632.698957</nRabsR>
-    </plugin>
+        <mQabsQ>-63</mQabsQ>
+        <nRabsR>-500</nRabsR>
+        <!-- <default_current>-0.05 -0.7 0.0</default_current> -->
+      </plugin>
     <!-- Publishes perfect odometry data for testing controllers -->
     <plugin
       filename="gz-sim-odometry-publisher-system"
       name="gz::sim::systems::OdometryPublisher">
-      <odom_frame>odom</odom_frame>
-      <robot_base_frame>base_link</robot_base_frame>
       <dimensions>3</dimensions>
     </plugin>

Commit message: Move sonoptix to top to match real vehicle

File: pontus_description/models/pontus/pontus.xacro (robot description, xacro)
@@ -97,5 +97,5 @@
   <!-- Forward Sonar -->
   <xacro:sonoptix_macro sonar_id="0">
-    <origin xyz="0.28 0 -0.15" rpy="${pi} ${10*pi/180} 0" />
+    <origin xyz="0.28 0 0.15" rpy="0 ${-5*pi/180} 0" />
   </xacro:sonoptix_macro>
   <!-- 360 Top Sonar -->

File: pontus_description/models/pontus/pontus_real.xacro (robot description, xacro)
@@ -88,5 +88,5 @@
   <!-- Forward Sonar -->
   <xacro:sonoptix_macro sonar_id="0">
-    <origin xyz="0.28 0 -0.15" rpy="0 ${10*pi/180} 0" />
+    <origin xyz="0.28 0 0.15" rpy="0 ${5*pi/180} 0" />
   </xacro:sonoptix_macro>
   <!-- 360 Top Sonar -->

Commit message: accidentally messed up sonoptix angle

File: pontus_description/models/pontus/pontus.xacro (robot description, xacro)
@@ -97,5 +97,5 @@
   <!-- Forward Sonar -->
   <xacro:sonoptix_macro sonar_id="0">
-    <origin xyz="0.28 0 0.15" rpy="0 ${-5*pi/180} 0" />
+    <origin xyz="0.28 0 0.15" rpy="0 ${5*pi/180} 0" />
   </xacro:sonoptix_macro>
   <!-- 360 Top Sonar -->

Commit message: Add vehicle params, remove unnecessary auv folders and launch files

File: pontus_description/models/pontus/pontus.xacro (robot description, xacro)
@@ -8,4 +8,8 @@
   <xacro:arg name="static" default="false"/>
   <xacro:property name="fluid_density" value="1025"/>
+  <xacro:property name="gravity" value="9.8"/>
+  <xacro:property name="thruster_max_thrust" value="52"/>
+  <xacro:property name="thruster_max_allowed" value="30"/>
+  <xacro:property name="thruster_min_allowed" value="2.6"/>
   <xacro:property name="namespace" value="pontus"/>
   <xacro:property name="mass" value="34.0194"/>
@@ -15,7 +19,19 @@
   <!-- Create pontus -->
   <link name="base_link">
+    <params
+      mass="${mass}"
+      length="${length}"
+      radius="${radius}"
+      diameter="${2*radius}"
+      volume="${volume}"
+      fluid_density="${fluid_density}"
+      gravity="${gravity}"
+      thruster_max_thrust="${thruster_max_thrust}"
+      thruster_max_allowed="${thruster_max_allowed}"
+      thruster_min_allowed="${thruster_min_allowed}"
+    />
     <inertial>
       <!-- This is calculated for slightly positive buoyancy -->
-      <mass value="${(volume * fluid_density) - 5.0}"/>
+      <mass value="${(volume * fluid_density) - 1.5}"/>
       <!-- TODO: insert actual calculations instead of precalculated value -->
       <inertia

Commit message: Add battery tubes and tweak controller

File: pontus_description/models/pontus/pontus.xacro (robot description, xacro)
@@ -4,6 +4,8 @@
   <xacro:include filename="$(find pontus_description)/models/pontus/components/sensors.xacro"/>
   <xacro:include filename="$(find pontus_description)/models/pontus/components/lights.xacro"/>
+  <xacro:include filename="$(find pontus_description)/models/pontus/components/battery_tubes.xacro"/>
   <!--<xacro:property name="mesh_file" value="file://$(find pontus_description)/models/pontus/meshes/pontus_body_mesh.STL"/>-->
   <xacro:arg name="sim" default="false"/>
+  <xacro:property name="sim" default="$(arg sim)"/>
   <xacro:arg name="static" default="false"/>
   <xacro:property name="fluid_density" value="1025"/>
@@ -13,8 +15,18 @@
   <xacro:property name="thruster_min_allowed" value="2.6"/>
   <xacro:property name="namespace" value="pontus"/>
-  <xacro:property name="mass" value="34.0194"/>
+  <xacro:property name="battery_tube_length" value="0.324"/>
+  <xacro:property name="battery_tube_radius" value="0.045"/>
+  <xacro:property name="battery_tube_volume" value="${pi*battery_tube_length*(battery_tube_radius**2)}"/>
   <xacro:property name="length" value="0.61"/>
   <xacro:property name="radius" value="0.1"/>
-  <xacro:property name="volume" value="${pi*length*(radius)**2}"/>
+  <xacro:property name="volume" value="${(pi*length*(radius**2)) + 2*battery_tube_volume}"/>
+  <xacro:if value="${sim == 'false'}">
+    <!-- Use the real vehicles mass -->
+    <xacro:property name="mass" value="34.0194"/>
+  </xacro:if>
+  <xacro:unless value="${sim == 'false'}">
+    <!-- Override the vehicle mass with one that will work well for sim-->
+    <xacro:property name="mass" value="${0.95 * (volume * fluid_density)}"/>
+  </xacro:unless>
   <!-- Create pontus -->
   <link name="base_link">
@@ -23,8 +35,10 @@
       length="${length}"
       radius="${radius}"
-      diameter="${2*radius}"
       volume="${volume}"
       fluid_density="${fluid_density}"
       gravity="${gravity}"
+      battery_tube_length="${battery_tube_length}"
+      battery_tube_radius="${battery_tube_radius}"
+      battery_tube_volume="${battery_tube_volume}"
       thruster_max_thrust="${thruster_max_thrust}"
       thruster_max_allowed="${thruster_max_allowed}"
@@ -33,6 +47,7 @@
     <inertial>
       <!-- This is calculated for slightly positive buoyancy -->
-      <mass value="${(volume * fluid_density) - 1.5}"/>
+      <mass value="${mass}"/>
       <!-- TODO: insert actual calculations instead of precalculated value -->
+      <!-- TODO: This also needs to be modified to account for the battery tubes -->
       <inertia
         ixx="55" ixy="0" ixz="0"
@@ -55,4 +70,6 @@
       </geometry>
     </collision>
+    <xacro:battery_tube_macro tube_id="0" length="0.324" radius="0.045" x="0.0" y="-0.1" z="0.13" />
+    <xacro:battery_tube_macro tube_id="1" length="0.324" radius="0.045" x="0.0" y="0.1" z="0.13" />
   </link>
   <!-- Thrusters -->
