Commit message: PONTUS DESCRIPTION FIX swaps the left and right sets of vertical thrusters to actually match what was intended

File: pontus_description/models/pontus/pontus.xacro (robot description, xacro)
@@ -76,17 +76,17 @@
   <!-- Back Left Vertical Thruster -->
   <xacro:T200_macro thruster_id="0">
-    <origin xyz="-0.075 -${radius + 0.07} 0" rpy="0 0 0" />
+    <origin xyz="-0.075 ${radius + 0.07} 0" rpy="0 0 0" />
   </xacro:T200_macro>
   <!-- Back Right Vertical Thruster -->
   <xacro:T200_macro thruster_id="1">
-    <origin xyz="-0.075 ${radius + 0.07} 0" rpy="0 0 ${180*pi/180}" />
+    <origin xyz="-0.075 -${radius + 0.07} 0" rpy="0 0 ${180*pi/180}" />
   </xacro:T200_macro>
   <!-- Front Left Vertical Thruster -->
   <xacro:T200_macro thruster_id="2">
-    <origin xyz="0.075 -${radius + 0.07} 0" rpy="0 0 0" />
+    <origin xyz="0.075 ${radius + 0.07} 0" rpy="0 0 0" />
   </xacro:T200_macro>
   <!-- Front Right Vertical Thruster -->
   <xacro:T200_macro thruster_id="3">
-    <origin xyz="0.075 ${radius + 0.07} 0" rpy="0 0 ${180*pi/180}" />
+    <origin xyz="0.075 -${radius + 0.07} 0" rpy="0 0 ${180*pi/180}" />
   </xacro:T200_macro>
   <!-- Back Left Horizontal Thruster -->

Commit message: fixing .xacro hardcoded frame ids for the cameras

File: pontus_description/models/pontus/pontus.xacro (robot description, xacro)
@@ -110,20 +110,18 @@
   </xacro:light_macro>
   <!-- Sensors -->
-  <!-- Forward Camera -->
-  <xacro:camera_macro camera_id="front">
+  <!-- Left Camera (forward-facing, port side) -->
+  <xacro:camera_macro camera_id="left">
     <origin xyz="0.305 0.075 0" rpy="0 0 0" />
   </xacro:camera_macro>
-  <xacro:camera_macro camera_id="3">
+  <!-- Right Camera (forward-facing, starboard side) -->
+  <xacro:camera_macro camera_id="right">
     <origin xyz="0.305 -0.075 0" rpy="0 0 0" />
   </xacro:camera_macro>
-  <!-- Side Camera -->
-  <xacro:camera_macro camera_id="4">
+  <!-- Tilted Down Camera (angled downward) -->
+  <xacro:camera_macro camera_id="tilted_down">
     <origin xyz="0 0.06 0.1" rpy="0 0 ${90*pi/180}" />
   </xacro:camera_macro>
-  <xacro:camera_macro camera_id="5">
-    <origin xyz="0 -0.06 0.1" rpy="0 0 -${90*pi/180}" />
-  </xacro:camera_macro>
-  <!-- Downward Camera -->
-  <xacro:camera_macro camera_id="1">
+  <!-- Facing Down Camera (pointing straight down) -->
+  <xacro:camera_macro camera_id="facing_down">
     <origin xyz="0 0 -0.1" rpy="0 ${90*pi/180} 0" />
   </xacro:camera_macro>
