Commit message: Tentative imu mounting transform

File: pontus_description/models/pontus/pontus.xacro (robot description, xacro)
@@ -142,5 +142,5 @@
   <!-- IMU -->
   <xacro:imu_macro imu_id="0">
-    <origin xyz="0 0 0" rpy="0 0 0" />
+    <origin xyz="0 0 0" rpy="0 ${-pi/2} ${pi/2}" />
   </xacro:imu_macro>
   <!-- Pressure -->

Commit message: Maybe working imu orientation calculation

File: pontus_description/models/pontus/pontus.xacro (robot description, xacro)
@@ -140,5 +140,6 @@
   <!-- IMU -->
   <xacro:imu_macro imu_id="0">
-    <origin xyz="0 0 0" rpy="0 ${-pi/2} ${pi/2}" />
+    <origin xyz="0 0 0" rpy="0 ${pi/2} 0" />
+    <!-- <origin xyz="0 0 0" rpy="${pi} 0 ${pi/2}" /> -->
   </xacro:imu_macro>
   <!-- Pressure -->
